Commit message: Fix wheel slippage

File: src/robot/description/robot_core.xacro (robot description, xacro)
@@ -61,5 +61,5 @@
         <collision>
             <geometry>
-                <cylinder radius="0.05" length="0.04"/>
+                <sphere radius="0.05"/>
             </geometry>
         </collision>
@@ -87,5 +87,5 @@
         <collision>
             <geometry>
-                <cylinder radius="0.05" length="0.04"/>
+                <sphere radius="0.05"/>
             </geometry>
         </collision>

Commit message: Integrate the SLAM Toolbox

File: src/robot/description/robot_core.xacro (robot description, xacro)
@@ -17,4 +17,12 @@
     <!-- Base Link -->
     <link name="base_link">
+    </link>
+    <!-- Base Footprint Link -->
+    <joint name="base_footprint_joint" type="fixed">
+        <parent link="base_link"/>
+        <child link="base_footprint"/>
+        <origin xyz="0 0 0" rpy="0 0 0"/>
+    </joint>
+    <link name="base_footprint">
     </link>
     <!-- Chassis -->
