Commit message: Change robot shape

File: src/robot/description/depth_camera.xacro (robot description, xacro)
@@ -4,5 +4,5 @@
         <parent link="chassis"/>
         <child link="camera_link"/>
-        <origin xyz="0.305 0 0.08" rpy="0 0 0"/>
+        <origin xyz="0.42 0 0.08" rpy="0 0 0"/>
     </joint>
     <link name="camera_link">
@@ -34,6 +34,6 @@
                 </image>
                 <clip>
-                    <near>0.05</near>
-                    <far>8.0</far>
+                    <near>0.42</near>
+                    <far>15.0</far>
                 </clip>
             </camera>

File: src/robot/description/lidar.xacro (robot description, xacro)
@@ -4,5 +4,5 @@
         <parent link="chassis"/>
         <child link="laser_frame"/>
-        <origin xyz="0.1 0 0.175" rpy="0 0 0"/>
+        <origin xyz="0.1 0 0.14" rpy="0 0 0"/>
     </joint>
     <link name="laser_frame">

File: src/robot/description/robot_core.xacro (robot description, xacro)
@@ -34,14 +34,14 @@
     <link name="chassis">
         <visual>
-            <origin xyz="0.15 0 0.075"/>
+            <origin xyz="0.17 0 0.06"/>
             <geometry>
-                <box size="0.3 0.3 0.15"/>
+                <cylinder radius="0.25" length="0.12"/>
             </geometry>
             <material name="orange"/>
         </visual>
         <collision>
-            <origin xyz="0.15 0 0.075"/>
+            <origin xyz="0.17 0 0.06"/>
             <geometry>
-                <box size="0.3 0.3 0.15"/>
+                <cylinder radius="0.25" length="0.12"/>
             </geometry>
         </collision>
@@ -109,5 +109,5 @@
         <parent link="chassis"/>
         <child link="caster_wheel"/>
-        <origin xyz="0.24 0 0"/>
+        <origin xyz="0.3 0 0"/>
     </joint>
     <link name="caster_wheel">
